Commit message: Fix joint interfaces in urdf

File: ackermann_vehicle_description/urdf/em_3905.urdf.xacro (robot description, xacro)
@@ -200,7 +200,8 @@
     <transmission name="${lr_prefix}_${fr_prefix}_shock_trans">
       <type>transmission_interface/SimpleTransmission</type>
-      <joint name="${lr_prefix}_${fr_prefix}_shock"/>
+      <joint name="${lr_prefix}_${fr_prefix}_shock">
+        <hardwareInterface>hardware_interface/EffortJointInterface</hardwareInterface>
+      </joint>
       <actuator name="${lr_prefix}_${fr_prefix}_shock_act">
-        <hardwareInterface>EffortJointInterface</hardwareInterface>
         <mechanicalReduction>1</mechanicalReduction>
       </actuator>
@@ -223,7 +224,8 @@
     <transmission name="${lr_prefix}_${fr_prefix}_axle_trans">
       <type>transmission_interface/SimpleTransmission</type>
-      <joint name="${lr_prefix}_${fr_prefix}_axle"/>
+      <joint name="${lr_prefix}_${fr_prefix}_axle">
+        <hardwareInterface>hardware_interface/EffortJointInterface</hardwareInterface>
+      </joint>
       <actuator name="${lr_prefix}_${fr_prefix}_axle_act">
-        <hardwareInterface>EffortJointInterface</hardwareInterface>
         <mechanicalReduction>1</mechanicalReduction>
       </actuator>
@@ -275,7 +277,8 @@
     <transmission name="${lr_prefix}_steering_trans">
       <type>transmission_interface/SimpleTransmission</type>
-      <joint name="${lr_prefix}_steering_joint"/>
+      <joint name="${lr_prefix}_steering_joint">
+        <hardwareInterface>hardware_interface/EffortJointInterface</hardwareInterface>
+      </joint>
       <actuator name="${lr_prefix}_steering_act">
-        <hardwareInterface>EffortJointInterface</hardwareInterface>
         <mechanicalReduction>1</mechanicalReduction>
       </actuator>

Commit message: Integrate stereo camera into model

File: ackermann_vehicle_description/urdf/em_3905.urdf.xacro (robot description, xacro)
@@ -28,4 +28,6 @@
 -->
 <robot name="em_3905" xmlns:xacro="http://www.ros.org/wiki/xacro">
+  <!-- includes -->
+  <xacro:include filename="$(find ackermann_vehicle_description)/urdf/stereo_camera.urdf.xacro" />
   <!-- Degree-to-radian conversions -->
   <xacro:property name="degrees_45" value="0.785398163"/>
@@ -35,5 +37,5 @@
   <xacro:property name="chassis_length" value="0.258"/>
   <xacro:property name="chassis_width" value="0.168"/>
-  <xacro:property name="chassis_height" value="0.01"/>
+  <xacro:property name="chassis_height" value="0.02"/>
   <xacro:property name="chassis_mass" value="2.788"/>
   <!-- battery_dist is the distance between the inner edges of the
@@ -298,15 +300,5 @@
   <!-- base_link must have geometry so that its axes can be displayed in
        rviz. -->
-  <link name="base_link">
-    <visual>
-      <geometry>
-        <box size="0.01 0.01 0.01"/>
-      </geometry>
-      <material name="chassis_mat"/>
-    </visual>
-  </link>
-  <gazebo reference="base_link">
-    <material>Gazebo/Grey</material>
-  </gazebo>
+  <link name="base_link" />
   <!-- Chassis -->
   <link name="chassis">
@@ -331,5 +323,5 @@
   </link>
   <gazebo reference="chassis">
-    <material>Gazebo/Grey</material>
+    <material>Gazebo/White</material>
   </gazebo>
   <joint name="base_link_to_chasis" type="fixed">
@@ -349,11 +341,32 @@
   <xacro:rear_wheel lr_prefix="right" fr_prefix="rear"
                     lr_reflect="-1" fr_reflect="-1"/>
+  <!-- camera mount -->
+  <link name="camera_mount">
+    <visual>
+      <geometry>
+        <cylinder radius="0.02" length="0.1" />
+      </geometry>
+      <material name="">
+      </material>
+    </visual>
+  </link>
+  <gazebo reference="camera_mount">
+    <material>Gazebo/Blue</material>
+  </gazebo>
+  <joint name="camera_mount_joint" type="fixed">
+    <parent link="chassis" />
+    <child link="camera_mount" />
+    <origin xyz="0.1 0.0 0.05" rpy="0 0 0" />
+  </joint>
+  <!-- camera -->
+  <xacro:stereo_camera parent="camera_mount" origin="0 0 0.06" />
+  <!-- gazebo plugins for control and odometry ground truth-->
   <gazebo>
-    <plugin name="gazebo_ros_control" filename="libgazebo_ros_control.so">
-      <!-- As of 10/7/13, setting controlPeriod to a value greater than
-           Gazebo's simulation period prevents the shock absorbers from
-           working.
-      <controlPeriod>${ctrl_period}</controlPeriod>
-      -->
+    <plugin name="gazebo_ros_control" filename="libgazebo_ros_control.so" />
+    <plugin name="gazebo_ros_p3d"     filename="libgazebo_ros_p3d.so">
+      <frameName>map</frameName>
+      <bodyName>base_link</bodyName>
+      <topicName>odom_truth</topicName>
+      <updateRate>30.0</updateRate>
     </plugin>
   </gazebo>

Commit message: mount vlp-16

File: ackermann_vehicle_description/urdf/em_3905.urdf.xacro (robot description, xacro)
@@ -1,33 +1,5 @@
 <?xml version="1.0"?>
-<!-- em_3905.urdf.xacro
-This file defines a model of a Traxxas(R) E-Maxx(R) #3905 RC (Radio Controlled)
-truck.
-Lengths are measured in meters, angles are measured in radians, and masses are
-measured in kilograms. All of these values are approximations.
-To work with Gazebo, each link must have an inertial element, even if
-the link only serves to connect two joints. To be visible in Gazebo, a link
-must have a collision element. Furthermore, the link must have a Gazebo
-material.
-Traxxas(R), E-Maxx(R), and Titan(R) are registered trademarks of Traxxas
-Management, LLC. em_3905.urdf.xacro was independently created by Wunderkammer
-Laboratory, and neither em_3905.urdf.xacro nor Wunderkammer Laboratory is
-affiliated with, sponsored by, approved by, or endorsed by Traxxas Management,
-LLC. Mabuchi Motor(R) is a registered trademark of Mabuchi Motor Co., Ltd.
-Corporation Japan. All other trademarks and service marks are the property of
-their respective owners.
-Copyright (c) 2011-2013 Wunderkammer Laboratory
-Licensed under the Apache License, Version 2.0 (the "License");
-you may not use this file except in compliance with the License.
-You may obtain a copy of the License at
-  http://www.apache.org/licenses/LICENSE-2.0
-Unless required by applicable law or agreed to in writing, software
-distributed under the License is distributed on an "AS IS" BASIS,
-WITHOUT WARRANTIES OR CONDITIONS OF ANY KIND, either express or implied.
-See the License for the specific language governing permissions and
-limitations under the License.
--->
-<robot name="em_3905" xmlns:xacro="http://www.ros.org/wiki/xacro">
+<robot name="ackermann_robot" xmlns:xacro="http://www.ros.org/wiki/xacro">
   <!-- includes -->
-  <xacro:include filename="$(find ackermann_vehicle_description)/urdf/stereo_camera.urdf.xacro" />
   <!-- Degree-to-radian conversions -->
   <xacro:property name="degrees_45" value="0.785398163"/>
@@ -35,20 +7,8 @@
   <!-- chassis_length is measured along the x axis, chassis_width
        along the y axis, and chassis_height along the z axis. -->
-  <xacro:property name="chassis_length" value="0.258"/>
-  <xacro:property name="chassis_width" value="0.168"/>
-  <xacro:property name="chassis_height" value="0.02"/>
-  <xacro:property name="chassis_mass" value="2.788"/>
-  <!-- battery_dist is the distance between the inner edges of the
-       batteries. battery_comp_depth is the battery compartment depth.
-       battery_length is measured along the x axis, battery_width
-       along the y axis, and battery_height along the z axis. -->
-  <xacro:property name="battery_x_offset" value="0.055"/>
-  <xacro:property name="battery_dist" value="0.065"/>
-  <xacro:property name="battery_comp_depth" value="0.02"/>
-  <xacro:property name="battery_comp_angle" value="0.34906585"/>
-  <xacro:property name="battery_length" value="0.16"/>
-  <xacro:property name="battery_width" value="0.047"/>
-  <xacro:property name="battery_height" value="0.024"/>
-  <xacro:property name="battery_mass" value="0.5025"/>
+  <xacro:property name="chassis_length" value="1"/>
+  <xacro:property name="chassis_width" value="0.75"/>
+  <xacro:property name="chassis_height" value="0.05"/>
+  <xacro:property name="chassis_mass" value="3.788"/>
   <!-- hub_dia and tire_dia are the diameters of the hub and tire,
        respectively. hex_hub_depth is the distance that the hex hub is
@@ -57,5 +17,5 @@
        axle_length. -->
   <xacro:property name="hub_dia" value="0.09652"/>
-  <xacro:property name="tire_dia" value="0.14605"/>
+  <xacro:property name="tire_dia" value="0.25"/>
   <xacro:property name="tire_width" value="0.0889"/>
   <xacro:property name="hex_hub_depth" value="0.01445"/>
@@ -65,6 +25,6 @@
        from a U joint to the corresponding hex hub. wheel_travel is the
        vertical wheel travel. -->
-  <xacro:property name="wheelbase" value="0.335"/>
-  <xacro:property name="hex_hub_dist" value="0.365"/>
+  <xacro:property name="wheelbase" value="1.02"/>
+  <xacro:property name="hex_hub_dist" value="1"/>
   <xacro:property name="axle_length" value="0.03"/>
   <xacro:property name="wheel_travel" value="0.084"/>
@@ -146,45 +106,4 @@
   </xacro:macro>
   <!-- Battery -->
-  <xacro:macro name="battery" params="prefix reflect">
-    <joint name="chassis_to_${prefix}_battery" type="fixed">
-      <parent link="chassis"/>
-      <child link="${prefix}_battery_offset"/>
-      <origin xyz="${battery_x_offset - battery_length / 2}
-                   ${reflect * battery_dist / 2}
-                   0"
-              rpy="${reflect * battery_comp_angle} 0 0"/>
-    </joint>
-    <link name="${prefix}_battery_offset">
-      <xacro:null_inertial/>
-    </link>
-    <joint name="offset_to_${prefix}_battery" type="fixed">
-      <parent link="${prefix}_battery_offset"/>
-      <child link="${prefix}_battery"/>
-      <origin xyz="0
-                   ${reflect * battery_width / 2}
-                   ${(battery_height / 2) - battery_comp_depth}"/>
-    </joint>
-    <link name="${prefix}_battery">
-      <visual>
-        <geometry>
-          <box size="${battery_length} ${battery_width} ${battery_height}"/>
-        </geometry>
-        <material name="battery_mat"/>
-      </visual>
-      <collision>
-        <geometry>
-          <box size="${battery_length} ${battery_width} ${battery_height}"/>
-        </geometry>
-      </collision>
-      <xacro:solid_cuboid_inertial
-         width="${battery_length}" depth="${battery_width}"
-         height="${battery_height}" mass="${battery_mass}">
-        <origin/>
-      </xacro:solid_cuboid_inertial>
-    </link>
-    <gazebo reference="${prefix}_battery">
-      <material>Gazebo/Blue</material>
-    </gazebo>
-  </xacro:macro>
   <!-- Shock absorber -->
   <xacro:macro name="shock"
@@ -329,7 +248,4 @@
     <child link="chassis"/>
   </joint>
-  <!-- Batteries -->
-  <xacro:battery prefix="left" reflect="1"/>
-  <xacro:battery prefix="right" reflect="-1"/>
   <!-- Wheels -->
   <xacro:front_wheel lr_prefix="left" fr_prefix="front"
@@ -341,24 +257,4 @@
   <xacro:rear_wheel lr_prefix="right" fr_prefix="rear"
                     lr_reflect="-1" fr_reflect="-1"/>
-  <!-- camera mount -->
-  <link name="camera_mount">
-    <visual>
-      <geometry>
-        <cylinder radius="0.02" length="0.1" />
-      </geometry>
-      <material name="">
-      </material>
-    </visual>
-  </link>
-  <gazebo reference="camera_mount">
-    <material>Gazebo/Blue</material>
-  </gazebo>
-  <joint name="camera_mount_joint" type="fixed">
-    <parent link="chassis" />
-    <child link="camera_mount" />
-    <origin xyz="0.1 0.0 0.05" rpy="0 0 0" />
-  </joint>
-  <!-- camera -->
-  <xacro:stereo_camera parent="camera_mount" origin="0 0 0.06" />
   <!-- gazebo plugins for control and odometry ground truth-->
   <gazebo>
@@ -371,3 +267,35 @@
     </plugin>
   </gazebo>
+  <link name="lidar_stand">
+    <visual>
+      <geometry>
+        <box size="0.1 0.1 0.7" />
+      </geometry>
+        <!--material name="black" /-->
+    </visual>
+    <collision>
+      <geometry>
+        <box size="0.1 0.1 0.7" />
+      </geometry>
+    </collision>
+    <inertial>
+      <mass value="1" />
+      <inertia ixx="0.145833" ixy="0.0" ixz="0.145833" iyy="0.0" iyz="0.0" izz="0.1250"/>
+    </inertial>
+  </link>
+  <joint name="joint_name" type="fixed">
+      <parent link="chassis"/>
+      <child link="lidar_stand"/>
+      <axis xyz="0.0 0.0 1.0"/>
+      <origin xyz="0.0 0.0 0.35"/>
+      <!--limit lower="0.0" upper="0.0" effort="0.0" velocity="0.0"/-->
+      <joint_properties damping="1.0" friction="1.0"/>
+  </joint>
+  <gazebo reference="lidar_stand">
+      <material>Gazebo/White</material>
+  </gazebo>
+  <xacro:include filename="$(find velodyne_description)/urdf/VLP-16.urdf.xacro"/>
+  <VLP-16 parent="chassis" name="velodyne" topic="/velodyne_points" hz="10" samples="1024" gpu="false" lasers="16" max_range="100">
+    <origin xyz="0 0 0.7" rpy="0 0 0 " />
+  </VLP-16>
 </robot>
